File: hardware/PUTM_DV_ASMC/PUTM_DV_ASMC.kicad_pcb (KiCad board)
At the start: 4 copper layers, 60 x 40 mm, 4 parts

Commit message: schematic without error
Parts:
- added C1: 100nF, Capacitor_SMD:C_0603_1608Metric_Pad1.08x0.95mm_HandSolder, F.Cu at (10.4, 107.4)
- added C13: 10u, Capacitor_SMD:C_0805_2012Metric_Pad1.18x1.45mm_HandSolder, F.Cu at (21.1, 58.2)
- added C14: 100n, Capacitor_SMD:C_0603_1608Metric_Pad1.08x0.95mm_HandSolder, F.Cu at (16.5, 57.9)
- added C15: 100n, Capacitor_SMD:C_0603_1608Metric_Pad1.08x0.95mm_HandSolder, F.Cu at (16.5, 60.4)
- added C16: 22u, Capacitor_SMD:CP_Elec_5x5.8, F.Cu at (27.9, 60.1)
- added C17: 22u, Capacitor_SMD:C_0805_2012Metric_Pad1.18x1.45mm_HandSolder, F.Cu at (21.1, 61.2)
- added C18: 10u, Capacitor_SMD:C_0805_2012Metric_Pad1.18x1.45mm_HandSolder, F.Cu at (21.1, 64.2)
- added C19: 22u, Capacitor_SMD:CP_Elec_5x5.8, F.Cu at (27.9, 66.9)
- added C2: 100n, Capacitor_SMD:C_0603_1608Metric, F.Cu at (29.0, 107.4)
- added C20: 10u, Capacitor_SMD:C_0805_2012Metric_Pad1.18x1.45mm_HandSolder, F.Cu at (21.1, 67.2)
- added C21: 22u, Capacitor_SMD:C_0805_2012Metric_Pad1.18x1.45mm_HandSolder, F.Cu at (21.1, 70.2)
- added C22: 100n, Capacitor_SMD:C_0603_1608Metric_Pad1.08x0.95mm_HandSolder, F.Cu at (16.5, 62.9)
- added C23: 100n, Capacitor_SMD:C_0603_1608Metric_Pad1.08x0.95mm_HandSolder, F.Cu at (16.5, 65.4)
- added C24: 22u, Capacitor_SMD:C_0805_2012Metric_Pad1.18x1.45mm_HandSolder, F.Cu at (21.1, 73.2)
- added C25: 22u, Capacitor_SMD:C_0805_2012Metric_Pad1.18x1.45mm_HandSolder, F.Cu at (21.1, 76.2)
- added C26: 22u, Capacitor_SMD:C_0805_2012Metric_Pad1.18x1.45mm_HandSolder, F.Cu at (21.1, 79.2)
- added C27: 100n, Capacitor_SMD:C_0603_1608Metric_Pad1.08x0.95mm_HandSolder, F.Cu at (64.8, 25.7)
- added C28: 100n, Capacitor_SMD:C_0603_1608Metric_Pad1.08x0.95mm_HandSolder, F.Cu at (64.8, 28.2)
- added C29: 10n, Capacitor_SMD:C_0603_1608Metric_Pad1.08x0.95mm_HandSolder, F.Cu at (64.8, 30.7)
- added C3: 100nF, Capacitor_SMD:C_0603_1608Metric_Pad1.08x0.95mm_HandSolder, F.Cu at (10.4, 109.9)
- added C30: 10n, Capacitor_SMD:C_0603_1608Metric_Pad1.08x0.95mm_HandSolder, F.Cu at (64.8, 33.2)
- added C31: 47u, Capacitor_SMD:C_0805_2012Metric_Pad1.18x1.45mm_HandSolder, F.Cu at (69.4, 25.9)
- added C32: 4.7nF/Y2, CAPC5728X280N:CAPC5728X280N, F.Cu at (184.6, 26.3)
- added C33: 47u, Capacitor_SMD:C_0805_2012Metric_Pad1.18x1.45mm_HandSolder, F.Cu at (69.4, 28.9)
- added C34: 4.7nF/Y2, CAPC5728X280N:CAPC5728X280N, F.Cu at (184.6, 30.8)
- added C35: 47u, Capacitor_SMD:C_0805_2012Metric_Pad1.18x1.45mm_HandSolder, F.Cu at (69.4, 31.9)
- added C36: 47u, Capacitor_SMD:C_0805_2012Metric_Pad1.18x1.45mm_HandSolder, F.Cu at (69.4, 34.9)
- added C37: 47u, Capacitor_SMD:C_0805_2012Metric_Pad1.18x1.45mm_HandSolder, F.Cu at (69.4, 37.9)
- added C38: 47u, Capacitor_SMD:C_0805_2012Metric_Pad1.18x1.45mm_HandSolder, F.Cu at (69.4, 41.0)
- added C39: 47u, Capacitor_SMD:C_0805_2012Metric_Pad1.18x1.45mm_HandSolder, F.Cu at (69.4, 44.0)
- added C4: 6p, Capacitor_SMD:C_0603_1608Metric_Pad1.08x0.95mm_HandSolder, F.Cu at (1.40, 132.8)
- added C40: 47u, Capacitor_SMD:C_0805_2012Metric_Pad1.18x1.45mm_HandSolder, F.Cu at (69.4, 47.0)
- added C41: 100n, Capacitor_SMD:C_0603_1608Metric_Pad1.08x0.95mm_HandSolder, F.Cu at (64.8, 35.7)
- added C42: 10n, Capacitor_SMD:C_0603_1608Metric_Pad1.08x0.95mm_HandSolder, F.Cu at (64.8, 38.2)
- added C43: 100n, Capacitor_SMD:C_0603_1608Metric_Pad1.08x0.95mm_HandSolder, F.Cu at (64.8, 40.7)
- added C44: 10n, Capacitor_SMD:C_0603_1608Metric_Pad1.08x0.95mm_HandSolder, F.Cu at (64.8, 43.2)
- added C45: 100n, Capacitor_SMD:C_0603_1608Metric_Pad1.08x0.95mm_HandSolder, F.Cu at (74.7, 57.9)
- added C46: 100n, Capacitor_SMD:C_0603_1608Metric_Pad1.08x0.95mm_HandSolder, F.Cu at (74.7, 60.4)
- added C47: 220p, Capacitor_SMD:C_0603_1608Metric_Pad1.08x0.95mm_HandSolder, F.Cu at (75.3, 102.3)
- added C48: 100n, Capacitor_SMD:C_0603_1608Metric_Pad1.08x0.95mm_HandSolder, F.Cu at (75.3, 104.8)
- added C49: 22n, Capacitor_SMD:C_0603_1608Metric_Pad1.08x0.95mm_HandSolder, F.Cu at (75.3, 107.3)
- added C50: 470n, Capacitor_SMD:C_0603_1608Metric_Pad1.08x0.95mm_HandSolder, F.Cu at (75.3, 109.8)
- added C51: 10n, Capacitor_SMD:C_0603_1608Metric_Pad1.08x0.95mm_HandSolder, F.Cu at (75.3, 112.3)
- added C52: 10n, Capacitor_SMD:C_0603_1608Metric_Pad1.08x0.95mm_HandSolder, F.Cu at (75.3, 114.9)
- added C53: 10n, Capacitor_SMD:C_0603_1608Metric_Pad1.08x0.95mm_HandSolder, F.Cu at (75.3, 117.4)
- added C54: 10n, Capacitor_SMD:C_0603_1608Metric_Pad1.08x0.95mm_HandSolder, F.Cu at (75.3, 119.9)
- added C55: 220p, Capacitor_SMD:C_0603_1608Metric_Pad1.08x0.95mm_HandSolder, F.Cu at (49.0, 102.2)
- added C56: 100n, Capacitor_SMD:C_0603_1608Metric_Pad1.08x0.95mm_HandSolder, F.Cu at (49.0, 104.7)
- added C57: 22n, Capacitor_SMD:C_0603_1608Metric_Pad1.08x0.95mm_HandSolder, F.Cu at (49.0, 107.2)
- added C58: 470n, Capacitor_SMD:C_0603_1608Metric_Pad1.08x0.95mm_HandSolder, F.Cu at (49.0, 109.7)
- added C59: 10n, Capacitor_SMD:C_0603_1608Metric_Pad1.08x0.95mm_HandSolder, F.Cu at (49.0, 112.2)
- added C60: 10n, Capacitor_SMD:C_0603_1608Metric_Pad1.08x0.95mm_HandSolder, F.Cu at (49.0, 114.8)
- added C61: 10n, Capacitor_SMD:C_0603_1608Metric_Pad1.08x0.95mm_HandSolder, F.Cu at (49.0, 117.3)
- added C62: 10n, Capacitor_SMD:C_0603_1608Metric_Pad1.08x0.95mm_HandSolder, F.Cu at (49.0, 119.8)
- added D1: LED, LED_SMD:LED_0603_1608Metric_Pad1.05x0.95mm_HandSolder, F.Cu at (11.4, 120.1)
- added D10: 1N4007, Diode_THT:D_DO-41_SOD81_P10.16mm_Horizontal, F.Cu at (88.2, 79.0)
- added D11: 40V/3A, Diode_SMD:D_SOD-123F, F.Cu at (88.9, 113.0)
- added D12: 40V/3A, Diode_SMD:D_SOD-123F, F.Cu at (62.6, 112.9)
- added D13: PESD5V0L2BT, Package_TO_SOT_SMD:SOT-23_Handsoldering, F.Cu at (17.5, 47.6)
- added D14: BZX84C5V6, Package_TO_SOT_SMD:SOT-23, F.Cu at (32.3, 47.3)
- added D15: BZX84C3V6-E3-08, Package_TO_SOT_SMD:SOT-23, F.Cu at (32.3, 51.8)
- added D16: PESD5V0L2BT, Package_TO_SOT_SMD:SOT-23_Handsoldering, F.Cu at (17.5, 52.4)
- added D17: 3.6V/400W, Package_TO_SOT_SMD:SOT-23-6, F.Cu at (37.3, 47.5)
- added D2: LED, LED_SMD:LED_0603_1608Metric_Pad1.05x0.95mm_HandSolder, F.Cu at (9.60, 120.2)
- added D3: LED, LED_SMD:LED_0603_1608Metric_Pad1.05x0.95mm_HandSolder, F.Cu at (7.60, 120.1)
- added D4: LED, LED_SMD:LED_0603_1608Metric_Pad1.05x0.95mm_HandSolder, F.Cu at (5.80, 120.1)
- added D5: 30V/200W, Diode_SMD:D_SOD-123, F.Cu at (40.5, 67.5)
- added D6: 9V1/200mW, Diode_SMD:D_SOD-323_HandSoldering, F.Cu at (26.0, 84.9)
- added D7: LED_+3V3, LED_SMD:LED_0603_1608Metric_Pad1.05x0.95mm_HandSolder, F.Cu at (20.9, 82.0)
- added D8: LED_+5V, LED_SMD:LED_0603_1608Metric_Pad1.05x0.95mm_HandSolder, F.Cu at (20.9, 84.6)
- added F1: 33V/1A5, Fuse:Fuse_2920_7451Metric_Pad2.10x5.45mm_HandSolder, F.Cu at (38.6, 73.9)
- added F2: 6V/1A, Fuse:Fuse_0805_2012Metric_Pad1.15x1.40mm_HandSolder, F.Cu at (43.3, 78.8)
- added F3: 6V/1A, Fuse:Fuse_0805_2012Metric_Pad1.15x1.40mm_HandSolder, F.Cu at (43.3, 81.8)
- added FB1: 2K@100MHz, Inductor_SMD:L_0805_2012Metric_Pad1.05x1.20mm_HandSolder, F.Cu at (19.4, 122.0)
- added FB2: 2K@100MHz, Inductor_SMD:L_0805_2012Metric_Pad1.05x1.20mm_HandSolder, F.Cu at (74.2, 25.8)
- added FB3: 2K@100MHz, Inductor_SMD:L_0805_2012Metric_Pad1.05x1.20mm_HandSolder, F.Cu at (74.2, 28.5)
- added FB4: 2K@100MHz, Inductor_SMD:L_0805_2012Metric_Pad1.05x1.20mm_HandSolder, F.Cu at (74.2, 31.3)
- added FB5: 2K@100MHz, Inductor_SMD:L_0805_2012Metric_Pad1.05x1.20mm_HandSolder, F.Cu at (74.2, 34.0)
- added FB6: 2K@100MHz, Inductor_SMD:L_0805_2012Metric_Pad1.05x1.20mm_HandSolder, F.Cu at (74.2, 36.8)
- added FB7: 2K@100MHz, Inductor_SMD:L_0805_2012Metric_Pad1.05x1.20mm_HandSolder, F.Cu at (74.2, 39.5)
- added FB8: 2K@100MHz, Inductor_SMD:L_0805_2012Metric_Pad1.05x1.20mm_HandSolder, F.Cu at (74.2, 42.3)
- added FB9: 2K@100MHz, Inductor_SMD:L_0805_2012Metric_Pad1.05x1.20mm_HandSolder, F.Cu at (74.2, 45.0)
- added H1: MountingHole_Pad_MP, MountingHole:MountingHole_4.3mm_M4_DIN965_Pad_TopOnly, F.Cu at (133.9, 60.6)
- added IC1: BTS722204ESAXUMA1, PDM:SOP65P600X115-25N, F.Cu at (90.4, 106.2)
- added IC2: BTS722204ESAXUMA1, PDM:SOP65P600X115-25N, F.Cu at (64.1, 106.1)
- added J1: FTSH-107-01-L-D-K, FTSH-107-XX-YYY-D-K:FTSH-107-XX-YYY-D-K, F.Cu at (41.8, 91.9)
- added J2: IPBS-110-01-XX-D-GP, PDM:IPBT110H1TDRAGP, F.Cu at (151.3, 61.0)
- added JP1: Jumper_2_Small_Bridged, Jumper:SolderJumper-2_P1.3mm_Open_TrianglePad1.0x1.5mm, F.Cu at (24.0, 122.3)
- added L1: 68u/1A4, Inductor_SMD:L_TDK_VLS6045EX_VLS6045AF, F.Cu at (37.1, 81.1)
- added Q1: 30V/5A, Package_TO_SOT_SMD:SOT-23-3, F.Cu at (35.0, 68.0)
- added R1: 1k, Resistor_SMD:R_0603_1608Metric, F.Cu at (29.0, 109.9)
- added R10: 1k, Resistor_SMD:R_0603_1608Metric_Pad0.98x0.95mm_HandSolder, F.Cu at (16.5, 70.5)
- added R11: 510k, Resistor_SMD:R_0603_1608Metric_Pad0.98x0.95mm_HandSolder, F.Cu at (16.5, 73.0)
- added R12: 13k3, Resistor_SMD:R_0603_1608Metric_Pad0.98x0.95mm_HandSolder, F.Cu at (16.5, 75.5)
- added R13: 100k, Resistor_SMD:R_0603_1608Metric_Pad0.98x0.95mm_HandSolder, F.Cu at (16.5, 78.0)
- added R14: 1k, Resistor_SMD:R_0603_1608Metric_Pad0.98x0.95mm_HandSolder, F.Cu at (16.5, 80.5)
- added R15: 100K, Resistor_SMD:R_0603_1608Metric_Pad0.98x0.95mm_HandSolder, F.Cu at (64.8, 45.7)
- added R16: 100K, Resistor_SMD:R_0603_1608Metric_Pad0.98x0.95mm_HandSolder, F.Cu at (64.8, 48.2)
- added R17: 2k, Resistor_SMD:R_0603_1608Metric_Pad0.98x0.95mm_HandSolder, F.Cu at (74.7, 62.9)
- added R18: 2k, Resistor_SMD:R_0603_1608Metric_Pad0.98x0.95mm_HandSolder, F.Cu at (74.7, 65.4)
- added R19: 10k, Resistor_SMD:R_0603_1608Metric_Pad0.98x0.95mm_HandSolder, F.Cu at (74.7, 67.9)
- added R2: 1K, Resistor_SMD:R_0603_1608Metric_Pad0.98x0.95mm_HandSolder, F.Cu at (11.4, 123.7)
- added R20: 10k, Resistor_SMD:R_0603_1608Metric_Pad0.98x0.95mm_HandSolder, F.Cu at (74.7, 70.5)
- added R21: 2.2k, Resistor_SMD:R_1206_3216Metric_Pad1.30x1.75mm_HandSolder, F.Cu at (89.3, 82.7)
- added R22: 100R, Resistor_SMD:R_0603_1608Metric, F.Cu at (84.3, 78.1)
- added R23: 100R, Resistor_SMD:R_0603_1608Metric, F.Cu at (84.3, 80.6)
- added R24: 10k, Resistor_SMD:R_0603_1608Metric, F.Cu at (84.3, 83.1)
- added R25: 10k, Resistor_SMD:R_0603_1608Metric, F.Cu at (84.3, 85.6)
- added R26: 100R, Resistor_SMD:R_0603_1608Metric, F.Cu at (16.3, 89.6)
- added R27: 10k, Resistor_SMD:R_0603_1608Metric, F.Cu at (16.3, 92.2)
- added R28: 100R, Resistor_SMD:R_0603_1608Metric, F.Cu at (16.3, 94.7)
- added R29: 10k, Resistor_SMD:R_0603_1608Metric, F.Cu at (16.3, 97.2)
- added R3: 1K, Resistor_SMD:R_0603_1608Metric_Pad0.98x0.95mm_HandSolder, F.Cu at (9.60, 123.7)
- added R30: 4k7, Resistor_SMD:R_0603_1608Metric_Pad0.98x0.95mm_HandSolder, F.Cu at (79.6, 102.3)
- added R31: 4k7, Resistor_SMD:R_0603_1608Metric_Pad0.98x0.95mm_HandSolder, F.Cu at (79.6, 104.8)
- added R32: 4k7, Resistor_SMD:R_0603_1608Metric_Pad0.98x0.95mm_HandSolder, F.Cu at (79.6, 107.3)
- added R33: 470R, Resistor_SMD:R_0603_1608Metric_Pad0.98x0.95mm_HandSolder, F.Cu at (79.6, 109.8)
- added R34: 330R, Resistor_SMD:R_0603_1608Metric_Pad0.98x0.95mm_HandSolder, F.Cu at (79.6, 112.3)
- added R35: 330R, Resistor_SMD:R_0603_1608Metric_Pad0.98x0.95mm_HandSolder, F.Cu at (79.6, 114.9)
- added R36: 330R, Resistor_SMD:R_0603_1608Metric_Pad0.98x0.95mm_HandSolder, F.Cu at (79.6, 117.4)
- added R37: 330R, Resistor_SMD:R_0603_1608Metric_Pad0.98x0.95mm_HandSolder, F.Cu at (79.6, 119.9)
- added R38: 10k, Resistor_SMD:R_0603_1608Metric_Pad0.98x0.95mm_HandSolder, F.Cu at (84.0, 102.3)
- added R39: 10k, Resistor_SMD:R_0603_1608Metric_Pad0.98x0.95mm_HandSolder, F.Cu at (84.0, 104.8)
- added R4: 1K, Resistor_SMD:R_0603_1608Metric_Pad0.98x0.95mm_HandSolder, F.Cu at (7.80, 123.7)
- added R40: 10k, Resistor_SMD:R_0603_1608Metric_Pad0.98x0.95mm_HandSolder, F.Cu at (84.0, 107.3)
- added R41: 10k, Resistor_SMD:R_0603_1608Metric_Pad0.98x0.95mm_HandSolder, F.Cu at (84.0, 109.8)
- added R42: 1k2, Resistor_SMD:R_0603_1608Metric_Pad0.98x0.95mm_HandSolder, F.Cu at (84.0, 112.3)
- added R43: 47R, Resistor_SMD:R_0603_1608Metric_Pad0.98x0.95mm_HandSolder, F.Cu at (84.0, 114.9)
- added R44: 4k7, Resistor_SMD:R_0603_1608Metric_Pad0.98x0.95mm_HandSolder, F.Cu at (53.3, 102.2)
- added R45: 4k7, Resistor_SMD:R_0603_1608Metric_Pad0.98x0.95mm_HandSolder, F.Cu at (53.3, 104.7)
- added R46: 4k7, Resistor_SMD:R_0603_1608Metric_Pad0.98x0.95mm_HandSolder, F.Cu at (53.3, 107.2)
- added R47: 470R, Resistor_SMD:R_0603_1608Metric_Pad0.98x0.95mm_HandSolder, F.Cu at (53.3, 109.7)
- added R48: 330R, Resistor_SMD:R_0603_1608Metric_Pad0.98x0.95mm_HandSolder, F.Cu at (53.3, 112.2)
- added R49: 330R, Resistor_SMD:R_0603_1608Metric_Pad0.98x0.95mm_HandSolder, F.Cu at (53.3, 114.8)
- added R5: 1K, Resistor_SMD:R_0603_1608Metric_Pad0.98x0.95mm_HandSolder, F.Cu at (6.00, 123.7)
- added R50: 330R, Resistor_SMD:R_0603_1608Metric_Pad0.98x0.95mm_HandSolder, F.Cu at (53.3, 117.3)
- added R51: 330R, Resistor_SMD:R_0603_1608Metric_Pad0.98x0.95mm_HandSolder, F.Cu at (53.3, 119.8)
- added R52: 10k, Resistor_SMD:R_0603_1608Metric_Pad0.98x0.95mm_HandSolder, F.Cu at (57.7, 102.2)
- added R53: 10k, Resistor_SMD:R_0603_1608Metric_Pad0.98x0.95mm_HandSolder, F.Cu at (57.7, 104.7)
- added R54: 10k, Resistor_SMD:R_0603_1608Metric_Pad0.98x0.95mm_HandSolder, F.Cu at (57.7, 107.2)
- added R55: 10k, Resistor_SMD:R_0603_1608Metric_Pad0.98x0.95mm_HandSolder, F.Cu at (57.7, 109.7)
- added R56: 1k2, Resistor_SMD:R_0603_1608Metric_Pad0.98x0.95mm_HandSolder, F.Cu at (57.7, 112.2)
- added R57: 47R, Resistor_SMD:R_0603_1608Metric_Pad0.98x0.95mm_HandSolder, F.Cu at (57.7, 114.8)
- added R6: 10k, Resistor_SMD:R_0603_1608Metric, F.Cu at (29.0, 112.4)
- added R7: 10k, Resistor_SMD:R_0603_1608Metric, F.Cu at (29.0, 114.9)
- added R8: 10k, Resistor_SMD:R_0603_1608Metric, F.Cu at (29.0, 117.4)
- added R9: 100k, Resistor_SMD:R_0603_1608Metric_Pad0.98x0.95mm_HandSolder, F.Cu at (16.5, 67.9)
- added T1: TP_VCC, TestPoint:TestPoint_Pad_1.0x1.0mm, F.Cu at (33.9, 58.2)
- added T2: TP_+5V, TestPoint:TestPoint_Pad_1.0x1.0mm, F.Cu at (33.9, 61.2)
- added T3: TP_+3V3, TestPoint:TestPoint_Pad_1.0x1.0mm, F.Cu at (33.9, 64.3)
- added T4: TP_GND, TestPoint:TestPoint_Pad_1.0x1.0mm, F.Cu at (37.0, 58.2)
- added T5: TP_GND, TestPoint:TestPoint_Pad_1.0x1.0mm, F.Cu at (37.0, 61.2)
- added T6: TP_VCC, TestPoint:TestPoint_Pad_1.0x1.0mm, F.Cu at (37.0, 64.3)
- added T7: TP_GND, TestPoint:TestPoint_Pad_1.0x1.0mm, F.Cu at (40.0, 58.2)
- added T8: TP_+5V, TestPoint:TestPoint_Pad_1.0x1.0mm, F.Cu at (40.0, 61.2)
- added T9: TP_GND, TestPoint:TestPoint_Pad_1.0x1.0mm, F.Cu at (40.0, 64.3)
- added TP1: TestPoint_Small, TestPoint:TestPoint_THTPad_D1.0mm_Drill0.5mm, F.Cu at (27.7, 122.1)
- added TP2: TestPoint_Small, TestPoint:TestPoint_Pad_D1.0mm, F.Cu at (93.8, 82.6)
- added TP6: TestPoint_Small, TestPoint:TestPoint_Pad_D1.0mm, F.Cu at (19.8, 89.9)
- added TP7: TestPoint_Small, TestPoint:TestPoint_Pad_D1.0mm, F.Cu at (19.8, 93.0)
- added U1: LM4040C33FTA, Package_TO_SOT_SMD:SOT-23, F.Cu at (19.4, 125.5)
- added U2: STM32G484RETx, Package_QFP:LQFP-64_10x10mm_P0.5mm, F.Cu at (9.40, 133.6)
- added U3: LM1117-3.3, Package_TO_SOT_SMD:SOT-223-3_TabPin2, F.Cu at (28.4, 74.5)
- added U4: TPS54202HDDCR, Package_TO_SOT_SMD:SOT-23-6_Handsoldering, F.Cu at (26.4, 81.1)
- added U5: ADM3057ExRW, Package_SO:SOIC-20W_7.5x12.8mm_P1.27mm, F.Cu at (83.2, 31.7)
- added U6: ADM3057ExRW, Package_SO:SOIC-20W_7.5x12.8mm_P1.27mm, F.Cu at (96.1, 31.7)
- added U8: TLP291-4, Package_SO:SOIC-16_4.55x10.3mm_P1.27mm, F.Cu at (67.2, 62.7)
- added Y1: ATX-11-F-32.000MHZ-F05-T, ATX11F32000MHZF05T:ATX11F32000MHZF05T, F.Cu at (39.0, 101.1)
- moved REF** 89.4 mm to (242.9, 134.0)
- moved REF** 89.4 mm to (192.9, 164.0)
- moved REF** 89.4 mm to (192.9, 134.0)
- moved REF** 89.4 mm to (242.9, 164.0)
Other:
- board size 60 x 40 mm -> 80 x 60 mm
- board text removed: "Template"
- board text removed: "v${REVISION}"
