File: hardware/PUTM_DV_ASMC/PUTM_DV_ASMC.kicad_pcb (KiCad board)
At the start: 4 copper layers, 88.4 x 88.2 mm, 184 parts, among them IC1 BTS722204ESAXUMA1, IC2 BTS722204ESAXUMA1, J1 FTSH-107-01-L-D-K, J2 IPBS-110-01-XX-D-GP, J4 74650073R, J5 74650073R, K2 FINDER-32.21-x000, Q1 30V/5A, Q2 BUK6D210, Q3 BUK6D210, Q4 BUK6D210, Q5 BUK6D210, T1 TP_VCC, T2 TP_+5V, T3 TP_+3V3, T4 TP_GND, T5 TP_GND, T6 TP_VCC, T7 TP_GND, T8 TP_+5V, T9 TP_GND, U1 LM4040C33FTA, U14 FODM217B, U15 FODM217B, U2 STM32G484RETx, U3 LM1117-3.3, U4 TPS54202HDDCR, U5 ADM3057ExRW, U6 ADM3057ExRW, Y1 ATX-11-F-32.000MHZ-F05-T

Commit message: work work work
Parts:
- removed T4, T7, T9: TP_GND, TestPoint:TestPoint_Pad_1.0x1.0mm
- removed TP1: TestPoint_Small, TestPoint:TestPoint_THTPad_D1.0mm_Drill0.5mm
- TP2, TP6, TP7: moved to B.Cu
- moved TP6 95.0 mm to (142.3, 66.7), turned to 180 degrees
- moved TP2 87.0 mm to (146.3, 66.8), turned to 180 degrees
- moved TP7 85.2 mm to (152.1, 68.5), turned to 180 degrees
- moved T1 32.1 mm to (203.1, 36.8)
- moved T8 29.2 mm to (207.0, 74.4)
- moved T5 20.5 mm to (206.6, 61.4)
- moved C23 3.93 mm to (200.9, 66.4), turned to 90 degrees
- moved D12 2.41 mm to (141.0, 94.0)
- moved C62 2.11 mm to (160.0, 40.3)
- moved D9 1.31 mm to (135.4, 44.0)
- moved R21 1.31 mm to (135.3, 48.6)
- moved R23 1.31 mm to (135.3, 58.4)
- moved R25 1.31 mm to (135.3, 56.6)
- moved Q3 1.31 mm to (135.3, 54.2)
- moved C1 1.21 mm to (167.0, 80.6)
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Connections:
- C2 pad 1: /Microcontroller/NRST -> /Connectors/NRST
- D11 pad 1: /Connectors/CAN2+ -> /CAN/CAN2_P
- D11 pad 2: /Connectors/CAN2- -> /CAN/CAN2_N
- D12 pad 1: /Connectors/CAN1+ -> /CAN/CAN1_P
- D12 pad 2: /Connectors/CAN1- -> /CAN/CAN1_N
- J1 pad 3: +3.3V -> +3V3
- J2 pad 17: /Connectors/CAN2+ -> /CAN/CAN2_P
- J2 pad 18: /Connectors/CAN2- -> /CAN/CAN2_N
- J2 pad 19: /Connectors/CAN1- -> /CAN/CAN1_N
- J2 pad 20: /Connectors/CAN1+ -> /CAN/CAN1_P
- JP1 pad 2: /Microcontroller/NRST -> /Connectors/NRST
- R6 pad 2: /Microcontroller/NRST -> /Connectors/NRST
- U2 pad 34: /Microcontroller/CAN2_RX -> /CAN/CAN2_RX
- U2 pad 35: /Microcontroller/CAN2_TX -> /CAN/CAN2_TX
- U2 pad 45: /Microcontroller/CAN1_RX -> /CAN/CAN1_RX
- U2 pad 46: /Microcontroller/CAN1_TX -> /CAN/CAN1_TX
- U2 pad 49: /Microcontroller/SWDIO -> /Connectors/SWDIO
- U2 pad 50: /Microcontroller/SWCLK -> /Connectors/SWCLK
- U2 pad 56: /Microcontroller/SWO -> /Connectors/SWO
- U2 pad 7: /Microcontroller/NRST -> /Connectors/NRST
- U5 pad 13: /CAN/CAN1- -> /CAN/CAN1_N
- U5 pad 14: /CAN/CAN1+ -> /CAN/CAN1_P
- U6 pad 13: /CAN/CAN2- -> /CAN/CAN2_N
- U6 pad 14: /CAN/CAN2+ -> /CAN/CAN2_P
Routing:
- net +5V: track 5.76 -> 82.8 mm
- net /DV_power_supply/SPI1.MOSI: track 0.00 -> 49.9 mm, vias 0 -> 4
- net /DV_power_supply/SPI1.NSS: track 0.00 -> 47.7 mm, vias 0 -> 3
- net /DV_power_supply/FUSE_IS0: track 2.22 -> 37.7 mm
- net /ASIS/ASSI_DI_PIN: track 0.00 -> 34.9 mm, vias 0 -> 2
- net /IO/BUZZER_PIN: track 0.00 -> 29.6 mm, vias 0 -> 2
- net /ASIS/ASSI_DO_PIN: track 0.00 -> 25.7 mm, vias 0 -> 2
- net /CAN/GND_CAN_ISO1: track 0.00 -> 25.5 mm
- net /DV_power_supply/LHI1: track 1.33 -> 23.5 mm, vias 0 -> 2
- net Net-(D10-A): track 5.26 -> 27.4 mm
- net GND: track 89.5 -> 111.0 mm, vias 100 -> 121
- net /DV_power_supply/SPI1.SCK: track 26.4 -> 45.6 mm, vias 2 -> 3
- net /DV_power_supply/SPI1.MISO: track 27.4 -> 45.5 mm, vias 0 -> 2
- net /CAN/GND_CAN_ISO2: track 0.00 -> 14.0 mm
- net Net-(U6-VISOIN): track 0.00 -> 11.4 mm
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- added copper zone on F.Cu, net /ASIS/ASSI_DI
- added copper zone on In1.Cu, net /ASIS/ASSI_DI
- added copper zone on In2.Cu, net /ASIS/ASSI_DI
- added copper zone on F.Cu, net /ASIS/ASSI_DO
- added copper zone on In1.Cu, net /ASIS/ASSI_DO
- added copper zone on In2.Cu, net /ASIS/ASSI_DO
- added copper zone on F.Cu, net /Connectors/OUT_BUZZER
- added copper zone on In1.Cu, net /Connectors/OUT_BUZZER
- added copper zone on In2.Cu, net /Connectors/OUT_BUZZER
- added copper zone on F.Cu, net Net-(D10-A)
- added copper zone on In1.Cu, net Net-(D10-A)
- added copper zone on In2.Cu, net Net-(D10-A)
- removed copper zone on B.Cu, net GND
