File: hardware/PUTM_DV_ASMC/PUTM_DV_ASMC.kicad_pcb (KiCad board)
At the start: 4 copper layers, 84.6 x 88.2 mm, 180 parts, among them IC1 BTS722204ESAXUMA1, IC2 BTS722204ESAXUMA1, J1 FTSH-107-01-L-D-K, J2 IPBS-110-01-XX-D-GP, J4 74650073R, J5 74650073R, K2 FINDER-32.21-x000, Q1 30V/5A, Q2 BUK6D210, Q3 BUK6D210, Q4 BUK6D210, Q5 BUK6D210, T1 TP_VCC, T2 TP_+5V, T3 TP_+3V3, T5 TP_GND, T6 TP_VCC, T8 TP_+5V, U1 LM4040C33FTA, U14 FODM217B, U15 FODM217B, U2 STM32G484RETx, U3 LM1117-3.3, U4 TPS54202HDDCR, U5 ADM3057ExRW, U6 ADM3057ExRW, Y1 ATX-11-F-32.000MHZ-F05-T

Commit message: pcb 99.5proc
Routing:
- removed copper zone on B.Cu, net /CAN/GND_CAN_ISO1
- removed copper zone on In1.Cu, net /CAN/GND_CAN_ISO1
- removed copper zone on In2.Cu, net /CAN/GND_CAN_ISO1
- removed copper zone on B.Cu, net /CAN/GND_CAN_ISO2
- removed copper zone on In1.Cu, net /CAN/GND_CAN_ISO2
- removed copper zone on In2.Cu, net /CAN/GND_CAN_ISO2
Changed lines of the file:
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@@
 		(capping no)
 		(filling no)
-		(zone_defaults)
 		(aux_axis_origin 116 116)
 		(grid_origin 116 116)
@@
 	)
 	(zone
-		(layers "F.Cu" "B.Cu" "In1.Cu" "In2.Cu")
+		(net "/CAN/GND_CAN_ISO2")
+		(layer "F.Cu")
 		(hatch edge 0.5)
+		(priority 13)
 		(connect_pads
-			(clearance 0)
+			(clearance 0.5)
 		)
 		(min_thickness 0.25)
-		(keepout
-			(tracks allowed)
-			(vias allowed)
-			(pads allowed)
-			(copperpour not_allowed)
-			(footprints allowed)
-		)
-		(placement
-			(enabled no)
-			(sheetname "")
-		)
-		(fill
+		(fill yes
 			(thermal_gap 0.5)
 			(thermal_bridge_width 0.5)
@@
 		(polygon
 			(pts
-				(xy 134 88.9) (xy 156.601967 88.80066) (xy 156.700108 107.983352) (xy 134.090365 108.089821)
+				(xy 187.6 89.1) (xy 187.686176 106.095107) (xy 167 106.2) (xy 166.9 89.2)
 			)
 		)
 	)
 	(zone
-		(net "/CAN/GND_CAN_ISO2")
-		(layers "F.Cu" "B.Cu" "In1.Cu" "In2.Cu")
+		(net "/CAN/GND_CAN_ISO1")
+		(layer "F.Cu")
 		(hatch edge 0.5)
 		(priority 13)
@@
 		(polygon
 			(pts
-				(xy 187.6 89.1) (xy 187.686176 106.095107) (xy 167 106.2) (xy 166.9 89.2)
+				(xy 156.107137 89.486974) (xy 156.2 106.5) (xy 135.5 106.6) (xy 135.4 89.6)
 			)
 		)
 	)
 	(zone
-		(net "/CAN/GND_CAN_ISO1")
 		(layers "F.Cu" "B.Cu" "In1.Cu" "In2.Cu")
 		(hatch edge 0.5)
-		(priority 13)
 		(connect_pads
-			(clearance 0.5)
+			(clearance 0)
 		)
 		(min_thickness 0.25)
-		(fill yes
+		(keepout
+			(tracks allowed)
+			(vias allowed)
+			(pads allowed)
+			(copperpour not_allowed)
+			(footprints allowed)
+		)
+		(placement
+			(enabled no)
+			(sheetname "")
+		)
+		(fill
 			(thermal_gap 0.5)
 			(thermal_bridge_width 0.5)
@@
 		(polygon
 			(pts
-				(xy 156.107137 89.486974) (xy 156.2 106.5) (xy 135.5 106.6) (xy 135.4 89.6)
+				(xy 147.289137 89.626221) (xy 156.551479 89.703071) (xy 156.563952 102.771043) (xy 147.18 102.78)
 			)
 		)
@@
 		(polygon
 			(pts
-				(xy 166.554768 88.494874) (xy 188.151106 88.399958) (xy 188.249247 107.58265) (xy 166.645133 107.684386)
+				(xy 178.493379 89.270245) (xy 187.755721 89.347095) (xy 187.768194 102.415067) (xy 178.384242 102.424024)
 			)
 		)
@@
 			)
 		)
+	)
+	(zone
+		(layers "B.Cu" "In1.Cu" "In2.Cu")
+		(hatch edge 0.5)
+		(connect_pads
+			(clearance 0)
+		)
+		(min_thickness 0.25)
+		(keepout
+			(tracks allowed)
+			(vias allowed)
+			(pads allowed)
+			(copperpour not_allowed)
+			(footprints allowed)
+		)
+		(placement
+			(enabled no)
+			(sheetname "")
+		)
+		(fill
+			(thermal_gap 0.5)
+			(thermal_bridge_width 0.5)
+			(island_removal_mode 0)
+		)
+		(polygon
+			(pts
+				(xy 134 88.9) (xy 156.601967 88.80066) (xy 156.700108 107.983352) (xy 134.090365 108.089821)
+			)
+		)
+	)
+	(zone
+		(layers "B.Cu" "In1.Cu" "In2.Cu")
+		(hatch edge 0.5)
+		(connect_pads
+			(clearance 0)
+		)
+		(min_thickness 0.25)
+		(keepout
+			(tracks allowed)
+			(vias allowed)
+			(pads allowed)
+			(copperpour not_allowed)
+			(footprints allowed)
+		)
+		(placement
+			(enabled no)
+			(sheetname "")
+		)
+		(fill
+			(thermal_gap 0.5)
+			(thermal_bridge_width 0.5)
+			(island_removal_mode 0)
+		)
+		(polygon
+			(pts
+				(xy 166.554768 88.494874) (xy 188.151106 88.399958) (xy 188.249247 107.58265) (xy 166.645133 107.684386)
+			)
+		)
