File: hardware/PUTM_DV_ASMC/PUTM_DV_ASMC.kicad_pcb (KiCad board)
At the start: 4 copper layers, 84.6 x 88.2 mm, 180 parts, among them IC1 BTS722204ESAXUMA1, IC2 BTS722204ESAXUMA1, J1 FTSH-107-01-L-D-K, J2 IPBS-110-01-XX-D-GP, J4 74650073R, J5 74650073R, K2 FINDER-32.21-x000, Q1 30V/5A, Q2 BUK6D210, Q3 BUK6D210, Q4 BUK6D210, Q5 BUK6D210, T1 TP_VCC, T2 TP_+5V, T3 TP_+3V3, T5 TP_GND, T6 TP_VCC, T8 TP_+5V, U1 LM4040C33FTA, U14 FODM217B, U15 FODM217B, U2 STM32G484RETx, U3 LM1117-3.3, U4 TPS54202HDDCR, U5 ADM3057ExRW, U6 ADM3057ExRW, Y1 ATX-11-F-32.000MHZ-F05-T

Commit message: pcb 100%
Routing:
- net /CAN/GND_CAN_ISO1: track 22.3 -> 28.5 mm, vias 7 -> 8
- net /CAN/GND_CAN_ISO2: track 25.3 -> 31.1 mm, vias 8 -> 9
- net Net-(C36-Pad1): track 10.3 -> 9.65 mm, vias 0 -> 2
- net Net-(C35-Pad1): track 10.2 -> 10.1 mm, vias 0 -> 2
