File: hardware/PUTM_DV_ASMC/PUTM_DV_ASMC.kicad_pcb (KiCad board)
At the start: 4 copper layers, 84.6 x 88.2 mm, 180 parts, among them IC1 BTS722204ESAXUMA1, IC2 BTS722204ESAXUMA1, J1 FTSH-107-01-L-D-K, J2 IPBS-110-01-XX-D-GP, J4 74650073R, J5 74650073R, K2 FINDER-32.21-x000, Q1 30V/5A, Q2 BUK6D210, Q3 BUK6D210, Q4 BUK6D210, Q5 BUK6D210, T1 TP_VCC, T2 TP_+5V, T3 TP_+3V3, T5 TP_GND, T6 TP_VCC, T8 TP_+5V, U1 LM4040C33FTA, U14 FODM217B, U15 FODM217B, U2 STM32G484RETx, U3 LM1117-3.3, U4 TPS54202HDDCR, U5 ADM3057ExRW, U6 ADM3057ExRW, Y1 ATX-11-F-32.000MHZ-F05-T

Commit message: update pcb layout
Parts:
- removed Q4, Q5: BUK6D210, UDFN2020-6:Diodes_UDFN2020-6_Type-F
- removed R26, R28: 100R, Resistor_SMD:R_0603_1608Metric
- removed R27, R29: 10k, Resistor_SMD:R_0603_1608Metric
- removed T5: TP_GND, TestPoint:TestPoint_Pad_1.0x1.0mm
- removed TP6, TP7: TestPoint_Small, TestPoint:TestPoint_Pad_D1.0mm
- added C70: 100n, Capacitor_SMD:C_0603_1608Metric_Pad1.08x0.95mm_HandSolder, F.Cu at (151.2, 62.8)
- added G***: LOGO, Logos:SignatureBox30mm, B.Cu at (144.5, 99.8)
- added Q6: BSS138, Package_TO_SOT_SMD:SOT-23, F.Cu at (147.1, 65.4)
- added R58: 10k, Resistor_SMD:R_0603_1608Metric, F.Cu at (152.2, 69.9)
- added R59: 47R, Resistor_SMD:R_0603_1608Metric, F.Cu at (153.2, 62.8)
- added R60: 100R, Resistor_SMD:R_0603_1608Metric, F.Cu at (146.2, 68.9)
- added R61: 10k, Resistor_SMD:R_0603_1608Metric, F.Cu at (147.9, 68.9)
- added R62: 560R, Resistor_SMD:R_0603_1608Metric, F.Cu at (148.6, 62.8)
- added R63: 100R, Resistor_SMD:R_0603_1608Metric, F.Cu at (145.5, 62.8)
- added U7: 74AHCT1G125, Package_TO_SOT_SMD:SOT-23-5, F.Cu at (152.2, 66.7)
- R21: value 2.2k -> 10k
- moved R22 4.70 mm to (141.6, 67.7)
- moved Q2 4.66 mm to (142.3, 64.4)
- moved R24 4.66 mm to (143.5, 67.5)
- moved TP2 3.31 mm to (143.4, 68.4)
- moved R5 0.15 mm to (181.0, 67.0)
- moved R6 0.08 mm to (159.0, 75.1)
Connections:
- J2 pad 4: /ASIS/ASSI_DO -> /ASIS/ASSI_OUT1
- J2 pad 5: /ASIS/ASSI_DI -> /ASIS/ASSI_OUT2
- R37 pad 1: /DV_power_supply/SPI1.NSS -> /DV_power_supply/SPI1.CSN1
- R51 pad 1: /DV_power_supply/SPI1.NSS -> /DV_power_supply/SPI1.CSN2
- U2 pad 38: /ASIS/ASSI_DO_PIN -> /ASIS/ASSI_SIG1
- U2 pad 39: /ASIS/ASSI_DI_PIN -> /ASIS/ASSI_SIG2
- U2 pad 42: /DV_power_supply/SPI1.NSS -> /DV_power_supply/SPI1.CSN1
- U2 pad 43: unconnected-(U2-PA9-Pad43) -> /DV_power_supply/SPI1.CSN2
Routing:
- net /ASIS/ASSI_DO: track 57.7 -> 0.00 mm, vias 2 -> 0
- net /ASIS/ASSI_OUT1: track 0.00 -> 52.7 mm, vias 0 -> 2
- net /ASIS/ASSI_DI: track 49.7 -> 0.00 mm, vias 1 -> 0
- net /DV_power_supply/SPI1.NSS: track 48.1 -> 0.00 mm, vias 3 -> 0
- net /ASIS/ASSI_OUT2: track 0.00 -> 44.8 mm, vias 0 -> 1
- net +5V: track 89.7 -> 130.2 mm, vias 4 -> 6
- net /ASIS/ASSI_DI_PIN: track 35.4 -> 0.00 mm, vias 2 -> 0
- net /DV_power_supply/SPI1.CSN2: track 0.00 -> 33.3 mm, vias 0 -> 2
- net /ASIS/ASSI_SIG2: track 0.00 -> 32.3 mm, vias 0 -> 2
- net /ASIS/ASSI_SIG1: track 0.00 -> 27.0 mm, vias 0 -> 2
- net /ASIS/ASSI_DO_PIN: track 26.3 -> 0.00 mm, vias 2 -> 0
- net /DV_power_supply/SPI1.CSN1: track 0.00 -> 23.6 mm, vias 0 -> 2
- net +3V3: track 45.7 -> 62.4 mm, vias 20 -> 23
- net /IO/BUZZER_PIN: track 30.0 -> 36.6 mm
- net Net-(Q4-G): track 4.31 -> 0.00 mm, vias 1 -> 0
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- removed copper zone on F.Cu, net /ASIS/ASSI_DI
- removed copper zone on In1.Cu, net /ASIS/ASSI_DI
- removed copper zone on In2.Cu, net /ASIS/ASSI_DI
- removed copper zone on F.Cu, net /ASIS/ASSI_DO
- removed copper zone on In1.Cu, net /ASIS/ASSI_DO
- removed copper zone on In2.Cu, net /ASIS/ASSI_DO
Other:
- board text added: "ASMC"
- board text added: "Michał Błotniak"
- board text added: "Reviewers: Piotr Witt Piotr Wojtczak"
- board text added: "v1.0"

Commit message: update pcb layout2
Parts:
- removed G***: LOGO, Logos:SignatureBox30mm
- moved C51 2.38 mm to (173.8, 39.1)
- moved C52 2.38 mm to (175.5, 39.1)
- moved C53 2.38 mm to (177.4, 39.1)
- moved C54 2.38 mm to (179.3, 39.1)
- moved C61 1.46 mm to (158.7, 38.9)
- moved C59 1.46 mm to (155.2, 38.9)
- moved C62 1.45 mm to (160.2, 38.9)
- moved C60 1.37 mm to (157.2, 38.9)
- moved C70 0.06 mm to (151.1, 62.8), turned to -90 degrees
Connections:
- C70 pad 1: +5V -> GND
- C70 pad 2: GND -> +5V
Routing:
- net /Connectors/ODRIVE4: track 12.3 -> 0.00 mm, vias 119 -> 114
- net /Connectors/OUT_RES: track 1.02 -> 4.78 mm
- net /Connectors/OUT_LIDAR: track 1.90 -> 4.61 mm
- net GND: track 168.4 -> 170.6 mm
- net /Connectors/OUT_EBS: track 3.37 -> 2.45 mm
- net +BATT: vias 0 -> 11
