File: hardware/PUTM_DV_ASMC/PUTM_DV_ASMC.kicad_pcb (KiCad board)
At the start: 4 copper layers, 84.6 x 88.2 mm, 180 parts, among them IC1 BTS722204ESAXUMA1, IC2 BTS722204ESAXUMA1, J1 FTSH-107-01-L-D-K, J2 IPBS-110-01-XX-D-GP, J4 74650073R, J5 74650073R, K2 FINDER-32.21-x000, Q1 30V/5A, Q2 BUK6D210, Q3 BUK6D210, Q6 BSS138, T1 TP_VCC, T2 TP_+5V, T3 TP_+3V3, T6 TP_VCC, T8 TP_+5V, U1 LM4040C33FTA, U14 FODM217B, U15 FODM217B, U2 STM32G484RETx, U3 LM1117-3.3, U4 TPS54202HDDCR, U5 ADM3057ExRW, U6 ADM3057ExRW, U7 74AHCT1G125, Y1 ATX-11-F-32.000MHZ-F05-T

Commit message: update pcb layout3 - before review
Parts:
- D11, D12: moved to B.Cu
- moved D11 68.9 mm to (135.8, 35.8)
- moved D12 58.5 mm to (130.7, 36.7), turned to -90 degrees
Routing:
- net /CAN/GND_CAN_ISO2: track 31.1 -> 135.3 mm, vias 9 -> 8
- net /CAN/GND_CAN_ISO1: track 28.5 -> 91.0 mm, vias 8 -> 7
- net /CAN/CAN2_P: track 122.1 -> 118.9 mm, vias 0 -> 1
- net /CAN/CAN2_N: track 121.5 -> 120.2 mm, vias 0 -> 1
- net /CAN/CAN1_P: track 81.6 -> 81.7 mm, vias 0 -> 1
- net /CAN/CAN1_N: vias 0 -> 1

Commit message: update pcb layout4 - before review
Routing:
- net +BATT: track 42.6 -> 44.7 mm, vias 11 -> 37

Commit message: update pcb layout5 - before review
Parts:
- JP1: value Jumper_2_Small_Bridged -> Jumper_Bridged
Connections:
- U2 pad 36: unconnected-(U2-PB14-Pad36) -> /IO/BUZZER_PIN
- U2 pad 37: /IO/BUZZER_PIN -> /ASIS/ASSI_SIG1
- U2 pad 38: /ASIS/ASSI_SIG1 -> unconnected-(U2-PC6-Pad38)
Changed lines of the file:
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@@
 			)
 		)
-		(property "Value" "Jumper_2_Small_Bridged"
+		(property "Value" "Jumper_Bridged"
 			(at 0 1.9 90)
 			(layer "F.Fab")
@@
 			(layers "F.Cu" "F.Mask" "F.Paste")
 			(roundrect_rratio 0.25)
-			(net "unconnected-(U2-PB14-Pad36)")
+			(net "/IO/BUZZER_PIN")
 			(pinfunction "PB14_36")
-			(pintype "bidirectional+no_connect")
+			(pintype "bidirectional")
 		)
 		(pad "37" smd roundrect
@@
 			(layers "F.Cu" "F.Mask" "F.Paste")
 			(roundrect_rratio 0.25)
-			(net "/IO/BUZZER_PIN")
+			(net "/ASIS/ASSI_SIG1")
 			(pinfunction "PB15_37")
 			(pintype "bidirectional")
@@
 			(layers "F.Cu" "F.Mask" "F.Paste")
 			(roundrect_rratio 0.25)
-			(net "/ASIS/ASSI_SIG1")
+			(net "unconnected-(U2-PC6-Pad38)")
 			(pinfunction "PC6_38")
 			(pintype "bidirectional")
@@
 	)
 	(segment
-		(start 171.4 75.3)
-		(end 172.15 74.55)
-		(width 0.2)
-		(layer "F.Cu")
-		(net "/IO/BUZZER_PIN")
-	)
-	(segment
 		(start 168.1 75.3)
 		(end 171.4 75.3)
@@
 	)
 	(segment
-		(start 172.15 74.55)
-		(end 173.225 74.55)
+		(start 171.65 75.05)
+		(end 171.4 75.3)
 		(width 0.2)
 		(layer "F.Cu")
@@
 		(net "/IO/BUZZER_PIN")
 	)
+	(segment
+		(start 173.225 75.05)
+		(end 171.65 75.05)
+		(width 0.2)
+		(layer "F.Cu")
+		(net "/IO/BUZZER_PIN")
+	)
 	(via
 		(at 168.1 75.3)
@@
 	)
 	(segment
-		(start 171.95 74.05)
-		(end 173.225 74.05)
+		(start 171.2 74.8)
+		(end 171.45 74.55)
 		(width 0.2)
 		(layer "F.Cu")
@@
 	)
 	(segment
-		(start 171.2 74.8)
-		(end 171.95 74.05)
+		(start 171.45 74.55)
+		(end 173.225 74.55)
 		(width 0.2)
 		(layer "F.Cu")

Commit message: update pcb layout after rewiev
Connections:
- U2 pad 12: /DV_power_supply/LHI0 -> /DV_power_supply/FUSE_IS0
- U2 pad 13: /DV_power_supply/LHI1 -> /DV_power_supply/FUSE_IS1
- U2 pad 40: /DV_power_supply/FUSE_IS0 -> /DV_power_supply/LHI1
- U2 pad 41: /DV_power_supply/FUSE_IS1 -> /DV_power_supply/LHI0
Routing:
- net +3V3: track 62.4 -> 72.8 mm, vias 23 -> 25
- net /CAN/GND_CAN_ISO1: track 91.0 -> 100.8 mm
- net /DV_power_supply/FUSE_IS1: track 39.1 -> 31.9 mm
- net +BATT: track 44.7 -> 38.8 mm, vias 37 -> 72
- net /DV_power_supply/LHI1: track 23.0 -> 27.6 mm
- net /DV_power_supply/LHI0: track 28.9 -> 24.7 mm
- net /CAN/GND_CAN_ISO2: track 135.3 -> 137.3 mm
- net /Connectors/UART_TX_PROG: track 22.0 -> 20.9 mm
- net /Connectors/SWO: track 30.9 -> 32.1 mm
- net /DV_power_supply/SPI1.SCK: track 45.6 -> 46.7 mm
- net /DV_power_supply/SPI1.CSN2: track 33.3 -> 32.4 mm
- net /DV_power_supply/SPI1.CSN1: track 23.6 -> 22.8 mm
- net /DV_power_supply/FUSE_IS0: track 41.4 -> 41.8 mm, vias 2 -> 4
