File: hardware/PUTM_DV_ASMC/DV_power_supply.kicad_sch (KiCad schematic)
At the start: 0 parts

Commit message: schematics without main connector
Other:
- added sheet Dv_power_supply_component (Dv_power_supply_component.kicad_sch)
- added sheet Odrive_power_supply (Odrive_power_supply.kicad_sch)
- title: (none) -> AS_power_controll

Commit message: done schematic v1
Changed lines of the file:
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@@
 		)
 	)
-	(global_label "ASSI_POWER"
-		(shape input)
+	(hierarchical_label "OUT_ASSI"
+		(shape output)
 		(at 241.3 69.85 0)
-		(fields_autoplaced yes)
-		(effects
-			(font
-				(size 1.27 1.27)
-			)
-			(justify left)
-		)
-		(property "Intersheetrefs" "${INTERSHEET_REFS}"
-			(at 255.8361 69.85 0)
-			(hide yes)
-			(show_name no)
-			(do_not_autoplace no)
-			(effects
-				(font
-					(size 1.27 1.27)
-				)
-				(justify left)
-			)
-		)
-	)
-	(global_label "RES_POWER"
-		(shape input)
+		(effects
+			(font
+				(size 1.27 1.27)
+			)
+			(justify left)
+		)
+	)
+	(hierarchical_label "OUT_LIDAR"
+		(shape output)
+		(at 241.3 59.69 0)
+		(effects
+			(font
+				(size 1.27 1.27)
+			)
+			(justify left)
+		)
+	)
+	(hierarchical_label "OUT_ODRIVE"
+		(shape output)
+		(at 151.13 62.23 0)
+		(effects
+			(font
+				(size 1.27 1.27)
+			)
+			(justify left)
+		)
+	)
+	(hierarchical_label "OUT_RES"
+		(shape output)
 		(at 241.3 54.61 0)
-		(fields_autoplaced yes)
-		(effects
-			(font
-				(size 1.27 1.27)
-			)
-			(justify left)
-		)
-		(property "Intersheetrefs" "${INTERSHEET_REFS}"
-			(at 255.3522 54.61 0)
-			(hide yes)
-			(show_name no)
-			(do_not_autoplace no)
-			(effects
-				(font
-					(size 1.27 1.27)
-				)
-				(justify left)
-			)
-		)
-	)
-	(global_label "LIDAR_POWER"
-		(shape input)
-		(at 241.3 59.69 0)
-		(fields_autoplaced yes)
-		(effects
-			(font
-				(size 1.27 1.27)
-			)
-			(justify left)
-		)
-		(property "Intersheetrefs" "${INTERSHEET_REFS}"
-			(at 256.9852 59.69 0)
-			(hide yes)
-			(show_name no)
-			(do_not_autoplace no)
-			(effects
-				(font
-					(size 1.27 1.27)
-				)
-				(justify left)
-			)
-		)
-	)
-	(global_label "ODRIVE_POWER"
-		(shape input)
-		(at 151.13 62.23 0)
-		(fields_autoplaced yes)
-		(effects
-			(font
-				(size 1.27 1.27)
-			)
-			(justify left)
-		)
-		(property "Intersheetrefs" "${INTERSHEET_REFS}"
-			(at 168.2666 62.23 0)
-			(hide yes)
-			(show_name no)
-			(do_not_autoplace no)
-			(effects
-				(font
-					(size 1.27 1.27)
-				)
-				(justify left)
-			)
-		)
-	)
-	(global_label "EBS_POWER"
-		(shape input)
-		(at 241.3 64.77 0)
-		(fields_autoplaced yes)
-		(effects
-			(font
-				(size 1.27 1.27)
-			)
-			(justify left)
-		)
-		(property "Intersheetrefs" "${INTERSHEET_REFS}"
-			(at 255.3522 64.77 0)
-			(hide yes)
-			(show_name no)
-			(do_not_autoplace no)
-			(effects
-				(font
-					(size 1.27 1.27)
-				)
-				(justify left)
-			)
+		(effects
+			(font
+				(size 1.27 1.27)
+			)
+			(justify left)
 		)
 	)
@@
 			)
 			(justify right)
+		)
+	)
+	(hierarchical_label "OUT_EBS"
+		(shape output)
+		(at 241.3 64.77 0)
+		(effects
+			(font
+				(size 1.27 1.27)
+			)
+			(justify left)
 		)
 	)
@@
 			)
 		)
-		(pin "OUTPUT_ODRIVE" input
+		(pin "OUTPUT_ODRIVE" output
 			(at 148.59 62.23 0)
 			(effects

Commit message: schematic without error
Other:
- sheet Odrive_power_supply ports: added ODRIVE[1..4]; removed OUTPUT_ODRIVE

Commit message: work on supply and zones
Changed lines of the file:
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@@
 		)
 	)
-	(label "SPI.MISO"
+	(label "SPI1.MISO"
 		(at 66.04 116.84 0)
 		(effects
@@
 		)
 	)
-	(label "LHI.0"
+	(label "LHI0"
 		(at 66.04 128.27 0)
 		(effects
@@
 		)
 	)
-	(label "SPI.NSS"
+	(label "FUSE_IS0"
+		(at 64.77 147.32 0)
+		(effects
+			(font
+				(size 1.27 1.27)
+			)
+			(justify left bottom)
+		)
+	)
+	(label "FUSE_IS1"
+		(at 64.77 149.86 0)
+		(effects
+			(font
+				(size 1.27 1.27)
+			)
+			(justify left bottom)
+		)
+	)
+	(label "SPI1.NSS"
 		(at 66.04 111.76 0)
 		(effects
@@
 		)
 	)
-	(label "SPI.MOSI"
+	(label "SPI1.MOSI"
 		(at 66.04 114.3 0)
 		(effects
@@
 		)
 	)
-	(label "LHI.1"
+	(label "LHI1"
 		(at 66.04 130.81 0)
 		(effects
@@
 		)
 	)
-	(label "SPI.SCK"
+	(label "SPI1.SCK"
 		(at 66.04 109.22 0)
 		(effects
@@
 		)
 	)
-	(hierarchical_label "SPI1_Bus{SPI}"
+	(hierarchical_label "SPI1{NSS SCK MISO MOSI}"
 		(shape bidirectional)
 		(at 57.15 95.25 180)
@@
 		)
 	)
-	(hierarchical_label "FUSE_ISO{FUSE_ISO.0 FUSE_ISO.1}"
+	(hierarchical_label "FUSE_IS[0..1]"
 		(shape output)
 		(at 58.42 139.7 180)
@@
 		)
 	)
-	(hierarchical_label "LHI{LHI.0 LHI.1}"
+	(hierarchical_label "LHI[0..1]"
 		(shape input)
 		(at 58.42 121.92 180)
