File: hardware/PUTM_DV_ASMC/DV_power_supply.kicad_sch (KiCad schematic)
At the start: 0 parts

Commit message: update spi schema
Other:
- sheet Dv_power_supply_component ports: added CSN2; removed NSS
- sheet Odrive_power_supply ports: added CSN1; removed NSS
