File: hardware/PUTM_DV_ASMC/IO.kicad_sch (KiCad schematic)
At the start: 22 parts, among them K2 FINDER-32.21-x000, Q2 BUK6D210, Q3 BUK6D210, U14 FODM217B, U15 FODM217B

Commit message: update spi schema
Parts:
- R21: value 2.2k -> 10k
Changed lines of the file:
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@@
 			)
 		)
-		(property "Value" "2.2k"
+		(property "Value" "10k"
 			(at 218.44 111.76 90)
 			(show_name no)

Commit message: edit footprint for diode before manufactur - now product version
Parts:
- D10: footprint Diode_SMD:D_0805_2012Metric_Pad1.15x1.40mm_HandSolder -> Diode_SMD:D_SOD-323_HandSoldering
Changed lines of the file:
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@@
 			)
 		)
-		(property "Footprint" "Diode_SMD:D_0805_2012Metric_Pad1.15x1.40mm_HandSolder"
+		(property "Footprint" "Diode_SMD:D_SOD-323_HandSoldering"
 			(at 161.29 123.19 90)
 			(hide yes)
