File: hardware/PUTM_DV_ASMC/Connectors.kicad_sch (KiCad schematic)
At the start: 7 parts, among them J1 FTSH-107-01-L-D-K, J2 IPBS-110-01-XX-D-GP, J4 74650073R, J5 74650073R

Commit message: work work work
Connections:
- net +3.3V renamed +3V3
- net CAN1+ renamed CAN1_P
- net CAN1- renamed CAN1_N
- net CAN2+ renamed CAN2_P
- net CAN2- renamed CAN2_N
Other:
- moved on the sheet: D12, J4

Commit message: can layout
Connections:
- net CAN2_N: now also J2.17; no longer J2.18
- net CAN2_P: now also J2.18; no longer J2.17
Changed lines of the file:
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@@
 		)
 	)
-	(label "CAN2_P"
+	(label "CAN2_N"
 		(at 132.08 50.8 180)
 		(effects
@@
 		)
 	)
-	(label "CAN2_N"
+	(label "CAN2_P"
 		(at 132.08 53.34 180)
 		(effects
