File: hardware/PUTM_DV_ASMC/Connectors.kicad_sch (KiCad schematic)
At the start: 7 parts, among them J1 FTSH-107-01-L-D-K, J2 IPBS-110-01-XX-D-GP, J4 74650073R, J5 74650073R

Commit message: update assi logic on schema and update .ioc
Connections:
- net ASSI_DI renamed ASSI_OUT2
- net ASSI_DO renamed ASSI_OUT1
Changed lines of the file:
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@@
 		)
 	)
-	(hierarchical_label "ASSI_DI"
+	(hierarchical_label "ASSI_OUT2"
 		(shape input)
 		(at 63.5 45.72 180)
@@
 		)
 	)
-	(hierarchical_label "ASSI_DO"
+	(hierarchical_label "ASSI_OUT1"
 		(shape input)
 		(at 63.5 43.18 180)

Commit message: after review2
Connections:
- net ADC is gone; now on net GND: J2.10
- net GPIO is gone; now on net GND: J2.2
