File: hardware/PUTM_DV_ASMC/Microcontroller.kicad_sch (KiCad schematic)
At the start: 28 parts, among them U1 LM4040C33FTA, U2 STM32G484RETx, Y1 ATX-11-F-32.000MHZ-F05-T

Commit message: update pcb after review
Connections:
- net CAN1_RX renamed CAN1-
- net CAN1_TX renamed CAN1+
- net CAN2_RX renamed CAN2-
- net CAN2_TX renamed CAN2+
Changed lines of the file:
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@@
 		)
 	)
-	(label "CAN1_RX"
+	(label "CAN1-"
 		(at 27.94 173.99 180)
 		(effects
@@
 		)
 	)
-	(label "CAN1_TX"
+	(label "CAN1+"
 		(at 27.94 177.8 180)
 		(effects
@@
 		)
 	)
-	(label "CAN2_TX"
+	(label "CAN2+"
 		(at 27.94 194.31 180)
 		(effects
@@
 		)
 	)
-	(label "CAN2_TX"
+	(label "CAN2+"
 		(at 251.46 132.08 180)
 		(effects
@@
 		)
 	)
-	(label "CAN2_RX"
+	(label "CAN2-"
 		(at 27.94 190.5 180)
 		(effects
@@
 		)
 	)
-	(label "CAN1_RX"
+	(label "CAN1-"
 		(at 251.46 83.82 180)
 		(effects
@@
 		)
 	)
-	(label "CAN1_TX"
+	(label "CAN1+"
 		(at 251.46 86.36 180)
 		(effects
@@
 		)
 	)
-	(label "CAN2_RX"
+	(label "CAN2-"
 		(at 251.46 129.54 180)
 		(effects
