File: hardware/PUTM_DV_ASMC/Microcontroller.kicad_sch (KiCad schematic)
At the start: 28 parts, among them U1 LM4040C33FTA, U2 STM32G484RETx, Y1 ATX-11-F-32.000MHZ-F05-T

Commit message: update assi logic on schema and update .ioc
Connections:
- net ASSI_DI_PIN renamed ASSI_SIG2_PIN
- net ASSI_DO_PIN renamed ASSI_SIG1_PIN
Changed lines of the file:
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@@
 		)
 	)
-	(hierarchical_label "ASSI_DO_PIN"
+	(hierarchical_label "ASSI_SIG1_PIN"
 		(shape output)
 		(at 175.26 93.98 180)
@@
 		)
 	)
-	(hierarchical_label "ASSI_DI_PIN"
-		(shape bidirectional)
+	(hierarchical_label "ASSI_SIG2_PIN"
+		(shape output)
 		(at 175.26 96.52 180)
 		(effects

Commit message: update spi schema
Connections:
- net SPI1.CSN2: now reaches U2.43 (PA9)
- net SPI1.NSS renamed SPI1.CSN1
- no-connect marks 18 -> 17
Changed lines of the file:
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@@
-	)
-	(no_connect
-		(at 233.68 78.74)
 	)
 	(no_connect
@@
 	)
 	(bus_entry
-		(at 102.87 138.43)
+		(at 95.25 139.7)
+		(size 2.54 -2.54)
+		(stroke
+			(width 0)
+			(type default)
+		)
+	)
+	(bus_entry
+		(at 95.25 137.16)
 		(size 2.54 -2.54)
 		(stroke
@@
 	)
 	(bus_entry
-		(at 102.87 135.89)
+		(at 95.25 134.62)
 		(size 2.54 -2.54)
 		(stroke
@@
 	)
 	(bus_entry
-		(at 102.87 133.35)
+		(at 95.25 132.08)
 		(size 2.54 -2.54)
 		(stroke
@@
 	)
 	(bus_entry
-		(at 102.87 130.81)
+		(at 95.25 129.54)
 		(size 2.54 -2.54)
 		(stroke
@@
 		)
 	)
+	(bus
+		(pts
+			(xy 97.79 129.54) (xy 97.79 127)
+		)
+		(stroke
+			(width 0)
+			(type default)
+		)
+	)
 	(wire
 		(pts
@@
 	(wire
 		(pts
+			(xy 87.63 139.7) (xy 95.25 139.7)
+		)
+		(stroke
+			(width 0)
+			(type default)
+		)
+	)
+	(wire
+		(pts
 			(xy 27.94 177.8) (xy 40.64 177.8)
 		)
@@
 	(wire
 		(pts
+			(xy 233.68 78.74) (xy 251.46 78.74)
+		)
+		(stroke
+			(width 0)
+			(type default)
+		)
+	)
+	(wire
+		(pts
 			(xy 52.07 78.74) (xy 43.18 78.74)
 		)
@@
 	(bus
 		(pts
-			(xy 105.41 135.89) (xy 105.41 125.73)
+			(xy 97.79 134.62) (xy 97.79 129.54)
 		)
 		(stroke
@@
 	(wire
 		(pts
-			(xy 86.36 135.89) (xy 102.87 135.89)
+			(xy 87.63 134.62) (xy 95.25 134.62)
 		)
 		(stroke
@@
 		)
 	)
-	(wire
-		(pts
-			(xy 86.36 130.81) (xy 102.87 130.81)
+	(bus
+		(pts
+			(xy 97.79 134.62) (xy 97.79 137.16)
+		)
+		(stroke
+			(width 0)
+			(type default)
+		)
+	)
+	(wire
+		(pts
+			(xy 87.63 129.54) (xy 95.25 129.54)
+		)
+		(stroke
+			(width 0)
+			(type default)
+		)
+	)
+	(bus
+		(pts
+			(xy 97.79 127) (xy 97.79 124.46)
 		)
 		(stroke
@@
 	(wire
 		(pts
-			(xy 86.36 138.43) (xy 102.87 138.43)
+			(xy 87.63 137.16) (xy 95.25 137.16)
 		)
 		(stroke
@@
 	(bus
 		(pts
-			(xy 105.41 125.73) (xy 107.95 125.73)
+			(xy 97.79 124.46) (xy 100.33 124.46)
 		)
 		(stroke
@@
 	(wire
 		(pts
-			(xy 86.36 133.35) (xy 102.87 133.35)
+			(xy 87.63 132.08) (xy 95.25 132.08)
 		)
 		(stroke
@@
 		)
 	)
-	(label "SPI1.SCK"
-		(at 86.36 138.43 180)
+	(label "SPI1.CSN2"
+		(at 251.46 78.74 180)
+		(effects
+			(font
+				(size 1.27 1.27)
+			)
+			(justify right bottom)
+		)
+	)
+	(label "SPI1.CSN1"
+		(at 87.63 137.16 180)
 		(effects
 			(font
@@
 		)
 	)
+	(label "SPI1.CSN2"
+		(at 87.63 139.7 180)
+		(effects
+			(font
+				(size 1.27 1.27)
+			)
+			(justify right bottom)
+		)
+	)
 	(label "DEBUG_LED_1"
 		(at 49.53 116.84 0)
@@
 	)
 	(label "SPI1.MISO"
-		(at 86.36 133.35 180)
-		(effects
-			(font
-				(size 1.27 1.27)
-			)
-			(justify right bottom)
-		)
-	)
-	(label "SPI1.NSS"
-		(at 86.36 135.89 180)
+		(at 87.63 132.08 180)
+		(effects
+			(font
+				(size 1.27 1.27)
+			)
+			(justify right bottom)
+		)
+	)
+	(label "SPI1.SCK"
+		(at 87.63 134.62 180)
 		(effects
 			(font
@@
 	)
 	(label "SPI1.MOSI"
-		(at 86.36 130.81 180)
+		(at 87.63 129.54 180)
 		(effects
 			(font
@@
 		)
 	)
-	(label "SPI1.NSS"
+	(label "SPI1.CSN1"
 		(at 251.46 76.2 180)
 		(effects
@@
 		)
 	)
-	(hierarchical_label "SPI1{NSS SCK MISO MOSI}"
+	(hierarchical_label "SPI1{CSN1 CSN2 SCK MISO MOSI}"
 		(shape bidirectional)
-		(at 107.95 125.73 0)
-		(effects
-			(font
+		(at 100.33 124.46 0)
+		(effects
+			(font

Commit message: update pcb layout4 - before review
Parts:
- JP1: value Jumper_2_Small_Bridged -> Jumper_Bridged
Other:
- moved on the sheet: C2, JP1, R6

Commit message: update pcb layout5 - before review
Connections:
- net ASSI_SIG1_PIN: now also U2.37 (PB15); no longer U2.38 (PC6)
- net BUZZER_PIN: now also U2.36 (PB14); no longer U2.37 (PB15)
- no-connect marks 17 -> 16
Changed lines of the file:
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@@
 	)
 	(no_connect
-		(at 233.68 134.62)
-	)
-	(no_connect
 		(at 233.68 81.28)
 	)
@@
 	(wire
 		(pts
+			(xy 233.68 134.62) (xy 256.54 134.62)
+		)
+		(stroke
+			(width 0)
+			(type default)
+		)
+	)
+	(wire
+		(pts
 			(xy 87.63 185.42) (xy 96.52 185.42)
 		)
@@
 	(wire
 		(pts
-			(xy 198.12 93.98) (xy 175.26 93.98)
-		)
-		(stroke
-			(width 0)
-			(type default)
-		)
-	)
-	(wire
-		(pts
 			(xy 29.21 137.16) (xy 25.4 137.16)
 		)
@@
 	(wire
 		(pts
-			(xy 233.68 137.16) (xy 256.54 137.16)
-		)
-		(stroke
-			(width 0)
-			(type default)
-		)
-	)
-	(wire
-		(pts
 			(xy 233.68 58.42) (xy 251.46 58.42)
 		)
@@
 	(wire
 		(pts
+			(xy 233.68 137.16) (xy 256.54 137.16)
+		)
+		(stroke
+			(width 0)
+			(type default)
+		)
+	)
+	(wire
+		(pts
 			(xy 233.68 106.68) (xy 251.46 106.68)
 		)
@@
 		)
 	)
+	(hierarchical_label "ASSI_SIG1_PIN"
+		(shape output)
+		(at 256.54 137.16 0)
+		(effects
+			(font
+				(size 1.27 1.27)
+			)
+			(justify left)
+		)
+	)
 	(hierarchical_label "STBY_CAN_1"
 		(shape output)
@@
 		)
 	)
-	(hierarchical_label "BUZZER_PIN"
-		(shape output)
-		(at 256.54 137.16 0)
-		(effects
-			(font
-				(size 1.27 1.27)
-			)
-			(justify left)
-		)
-	)
-	(hierarchical_label "ASSI_SIG1_PIN"
-		(shape output)
-		(at 175.26 93.98 180)
-		(effects
-			(font
-				(size 1.27 1.27)
-			)
-			(justify right)
-		)
-	)
 	(hierarchical_label "FUSE_IS[0..1]"
 		(shape input)
@@
 		)
 	)
+	(hierarchical_label "BUZZER_PIN"
+		(shape output)
+		(at 256.54 134.62 0)
+		(effects
+			(font
+				(size 1.27 1.27)
+			)
+			(justify left)
+		)
+	)

Commit message: update pcb layout after rewiev
Connections:
- net FUSE_IS0: now also U2.12 (PA0); no longer U2.40 (PC8)
- net FUSE_IS1: now also U2.13 (PA1); no longer U2.41 (PC9)
- net LHI0: now also U2.41 (PC9); no longer U2.12 (PA0)
- net LHI1: now also U2.40 (PC8); no longer U2.13 (PA1)
Changed lines of the file:
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@@
 	(wire
 		(pts
+			(xy 251.46 58.42) (xy 233.68 58.42)
+		)
+		(stroke
+			(width 0)
+			(type default)
+		)
+	)
+	(wire
+		(pts
 			(xy 27.94 177.8) (xy 40.64 177.8)
 		)
@@
 	(wire
 		(pts
-			(xy 180.34 99.06) (xy 198.12 99.06)
-		)
-		(stroke
-			(width 0)
-			(type default)
-		)
-	)
-	(wire
-		(pts
 			(xy 114.3 41.91) (xy 118.11 41.91)
 		)
@@
 		)
 	)
+	(wire
+		(pts
+			(xy 233.68 55.88) (xy 251.46 55.88)
+		)
+		(stroke
+			(width 0)
+			(type default)
+		)
+	)
 	(bus
 		(pts
@@
 	(wire
 		(pts
-			(xy 233.68 55.88) (xy 251.46 55.88)
+			(xy 198.12 99.06) (xy 180.34 99.06)
 		)
 		(stroke
@@
 	(wire
 		(pts
+			(xy 198.12 101.6) (xy 180.34 101.6)
+		)
+		(stroke
+			(width 0)
+			(type default)
+		)
+	)
+	(wire
+		(pts
 			(xy 38.1 35.56) (xy 38.1 34.29)
 		)
@@
 	(wire
 		(pts
-			(xy 233.68 58.42) (xy 251.46 58.42)
-		)
-		(stroke
-			(width 0)
-			(type default)
-		)
-	)
-	(wire
-		(pts
 			(xy 198.12 106.68) (xy 180.34 106.68)
 		)
@@
 	(wire
 		(pts
-			(xy 180.34 101.6) (xy 198.12 101.6)
-		)
-		(stroke
-			(width 0)
-			(type default)
-		)
-	)
-	(wire
-		(pts
 			(xy 87.63 88.9) (xy 104.14 88.9)
 		)
@@
 		)
 	)
-	(label "FUSE_IS0"
-		(at 180.34 99.06 0)
-		(effects
-			(font
-				(size 1.27 1.27)
-			)
-			(justify left bottom)
-		)
-	)
 	(label "CAN1-"
 		(at 27.94 173.99 180)
@@
 		)
 	)
-	(label "FUSE_IS1"
-		(at 180.34 101.6 0)
-		(effects
-			(font
-				(size 1.27 1.27)
-			)
-			(justify left bottom)
-		)
-	)
 	(label "CAN2+"
 		(at 27.94 194.31 180)
@@
 		)
 	)
-	(label "CAN2-"
-		(at 27.94 190.5 180)
+	(label "FUSE_IS0"
+		(at 251.46 55.88 180)
 		(effects
 			(font
@@
 		)
 	)
-	(label "LHI1"
-		(at 251.46 58.42 180)
+	(label "CAN2-"
+		(at 27.94 190.5 180)
 		(effects
 			(font
@@
 		)
 	)
-	(label "LHI0"
-		(at 251.46 55.88 180)
+	(label "LHI1"
+		(at 180.34 99.06 0)
 		(effects
 			(font
 				(size 1.27 1.27)
 			)
-			(justify right bottom)
+			(justify left bottom)
 		)
 	)
@@
 		)
 	)
+	(label "FUSE_IS1"
+		(at 251.46 58.42 180)
+		(effects
+			(font
+				(size 1.27 1.27)
+			)
+			(justify right bottom)
+		)
+	)
 	(label "CAN2-"
 		(at 251.46 129.54 180)
@@
 		)
 	)
+	(label "LHI0"
+		(at 180.34 101.6 0)
+		(effects
+			(font
+				(size 1.27 1.27)
+			)
+			(justify left bottom)
+		)
+	)
 	(hierarchical_label "STBY_CAN_2"
 		(shape output)
@@
 		)
 		(pin "24"
+			(alternate "ADC3_IN12")
 		)
 		(pin "41"
@@
 		)
 		(pin "43"
-			(alternate "USART1_TX")
 		)
 		(pin "7"

Commit message: after review2
Parts:
- removed Y1: ATX-11-F-32.000MHZ-F05-T, ATX11F32000MHZF05T:ATX11F32000MHZF05T, symbol Samacsys:ATX-11-F-32.000MHZ-F05-T
- added Y1: ECS-TXO-2520-33-320-AN-TR, ECS_TXO_2520_33_320_AN_TR:OSC_ECS-TXO-2520-33-320-AN-TR, symbol ECS_TXO_2520_33_320_AN_TR:ECS-TXO-2520-33-320-AN-TR
- C3: value 100nF -> 1nF
Connections:
- net +3V3: now also Y1.4 (VDD)
- net GND: now also Y1.1 (TRI-STATE), Y1.2 (GND)
- net HS_IN: now also Y1.3 (OUTPUT)
- net ADC: no longer names the net of U2.24 (PB0)
- net GPIO: no longer names the net of U2.25 (PB1)
- no-connect marks 16 -> 19
Other:
- note added: "MCU"
- moved on the sheet: C63, C64, C65, C66, C67, C68, C69, FB10, R7, R8, U2
