File: hardware/PUTM_DV_ASMC/Power_supply.kicad_sch (KiCad schematic)
At the start: 36 parts, among them Q1 30V/5A, T1 TP_VCC, T2 TP_+5V, T3 TP_+3V3, T6 TP_VCC, T8 TP_+5V, U3 LM1117-3.3, U4 TPS54202HDDCR

Commit message: update assi logic on schema and update .ioc
Changed lines of the file:
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@@
-	)
-	(junction
-		(at 85.09 127)
-		(diameter 0)
-		(color 0 0 0 0)
 	)
 	(junction
@@
 	(wire
 		(pts
-			(xy 85.09 124.46) (xy 85.09 127)
+			(xy 85.09 124.46) (xy 85.09 129.54)
 		)
 		(stroke
@@
 		(pts
 			(xy 105.41 153.67) (xy 105.41 157.48)
-		)
-		(stroke
-			(width 0)
-			(type default)
-		)
-	)
-	(wire
-		(pts
-			(xy 85.09 127) (xy 85.09 129.54)
 		)
 		(stroke
@@
 					(unit 1)
 				)
-			)
-		)
-	)
-	(symbol
-		(lib_id "power:PWR_FLAG")
-		(at 85.09 127 90)
-		(mirror x)
-		(unit 1)
-		(body_style 1)
-		(exclude_from_sim no)
-		(in_bom yes)
-		(on_board yes)
-		(in_pos_files yes)
-		(dnp no)
-		(property "Reference" "#FLG02"
-			(at 83.185 127 0)
-			(hide yes)
-			(show_name no)
-			(do_not_autoplace no)
-			(effects
-				(font
-					(size 1.27 1.27)
-				)
-			)
-		)
-		(property "Value" "3V3_FLAG"
-			(at 81.28 126.9999 90)
-			(show_name no)
-			(do_not_autoplace no)
-			(effects
-				(font
-					(size 1.27 1.27)
-				)
-				(justify left)
-			)
-		)
-		(property "Footprint" ""
-			(at 85.09 127 0)
-			(hide yes)
-			(show_name no)
-			(do_not_autoplace no)
-			(effects
-				(font
-					(size 1.27 1.27)
-				)
-			)
-		)
-		(property "Datasheet" ""
-			(at 85.09 127 0)
-			(hide yes)
-			(show_name no)
-			(do_not_autoplace no)
-			(effects
-				(font
-					(size 1.27 1.27)
-				)
-			)
-		)
-		(property "Description" "Special symbol for telling ERC where power comes from"
-			(at 85.09 127 0)
-			(hide yes)
-			(show_name no)
-			(do_not_autoplace no)
-			(effects
-				(font
-					(size 1.27 1.27)
-				)
-			)
-		)
-		(pin "1"
-		)
-		(instances
-			(project "PUTM_DV_ASMC"
-				(path "/b652b05a-4e3d-4ad1-b032-18886abe7d45/76c3c659-a748-4932-81b3-d10dc40d628f"
-					(reference "#FLG02")
-					(unit 1)
-				)
