File: hardware/PUTM_DV_ASMC/PUTM_DV_ASMC.kicad_sch (KiCad schematic)
At the start: 0 parts

Commit message: update assi logic on schema and update .ioc
Other:
- sheet ASIS ports: added ASSI_OUT1, ASSI_OUT2, ASSI_SIG1, ASSI_SIG2; removed ASSI_DI, ASSI_DI_PIN, ASSI_DO, ASSI_DO_PIN
- sheet Connectors ports: added ASSI_OUT1, ASSI_OUT2; removed ASSI_DI, ASSI_DO
- sheet Microcontroller ports: added ASSI_SIG1_PIN, ASSI_SIG2_PIN; removed ASSI_DI_PIN, ASSI_DO_PIN
Changed lines of the file:
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@@
-			)
-		)
-		(pin "ASSI_DI" input
-			(at 237.49 27.94 180)
-			(effects
-				(font
-					(size 1.27 1.27)
-				)
-				(justify left)
-			)
-		)
-		(pin "ASSI_DO" input
-			(at 237.49 30.48 180)
-			(effects
-				(font
-					(size 1.27 1.27)
-				)
-				(justify left)
 			)
 		)
@@
 		(pin "{CAN1}" bidirectional
 			(at 237.49 78.74 180)
+			(effects
+				(font
+					(size 1.27 1.27)
+				)
+				(justify left)
+			)
+		)
+		(pin "ASSI_OUT1" input
+			(at 237.49 27.94 180)
+			(effects
+				(font
+					(size 1.27 1.27)
+				)
+				(justify left)
+			)
+		)
+		(pin "ASSI_OUT2" input
+			(at 237.49 30.48 180)
 			(effects
 				(font
@@
 			)
 		)
-		(pin "ASSI_DI" output
+		(pin "ASSI_OUT1" output
 			(at 210.82 27.94 0)
 			(effects
@@
 			)
 		)
-		(pin "ASSI_DI_PIN" input
+		(pin "ASSI_OUT2" output
+			(at 210.82 30.48 0)
+			(effects
+				(font
+					(size 1.27 1.27)
+				)
+				(justify right)
+			)
+		)
+		(pin "ASSI_SIG1" input
 			(at 166.37 27.94 180)
 			(effects
@@
 			)
 		)
-		(pin "ASSI_DO" output
-			(at 210.82 30.48 0)
-			(effects
-				(font
-					(size 1.27 1.27)
-				)
-				(justify right)
-			)
-		)
-		(pin "ASSI_DO_PIN" input
+		(pin "ASSI_SIG2" input
 			(at 166.37 30.48 180)
 			(effects
@@
 			)
 		)
-		(pin "ASSI_DI_PIN" bidirectional
-			(at 144.78 27.94 0)
-			(effects
-				(font
-					(size 1.27 1.27)
-				)
-				(justify right)
-			)
-		)
-		(pin "ASSI_DO_PIN" output
-			(at 144.78 30.48 0)
-			(effects
-				(font
-					(size 1.27 1.27)
-				)
-				(justify right)
-			)
-		)
 		(pin "AS_SENSE_PIN" input
 			(at 144.78 128.27 0)
@@
 			(effects
 				(font
+					(size 1.27 1.27)
+				)
+				(justify right)
+			)
+		)
+		(pin "ASSI_SIG1_PIN" output
+			(at 144.78 27.94 0)
+			(effects
+				(font
+					(size 1.27 1.27)
+				)
+				(justify right)
+			)
+		)
+		(pin "ASSI_SIG2_PIN" output
+			(at 144.78 30.48 0)
+			(effects
+				(font

Commit message: update spi schema
Other:
- sheet DV_power_supply ports: added SPI1{CSN1 CSN2 SCK MISO MOSI}; removed SPI1{NSS SCK MISO MOSI}
- sheet Microcontroller ports: added SPI1{CSN1 CSN2 SCK MISO MOSI}; removed SPI1{NSS SCK MISO MOSI}
Changed lines of the file:
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@@
-			)
-		)
-		(pin "SPI1{NSS SCK MISO MOSI}" bidirectional
-			(at 166.37 44.45 180)
-			(effects
-				(font
-					(size 1.27 1.27)
-				)
-				(justify left)
 			)
 		)
@@
 		(pin "LHI[0..1]" input
 			(at 166.37 50.8 180)
+			(effects
+				(font
+					(size 1.27 1.27)
+				)
+				(justify left)
+			)
+		)
+		(pin "SPI1{CSN1 CSN2 SCK MISO MOSI}" bidirectional
+			(at 166.37 44.45 180)
 			(effects
 				(font
@@
 			)
 		)
-		(pin "SPI1{NSS SCK MISO MOSI}" bidirectional
-			(at 144.78 44.45 0)
-			(effects
-				(font
-					(size 1.27 1.27)
-				)
-				(justify right)
-			)
-		)
 		(pin "FUSE_IS[0..1]" input
 			(at 144.78 57.15 0)
@@
 			(effects
 				(font
+					(size 1.27 1.27)
+				)
+				(justify right)
+			)
+		)
+		(pin "SPI1{CSN1 CSN2 SCK MISO MOSI}" bidirectional
+			(at 144.78 44.45 0)
+			(effects
+				(font
