File: hardware/PUTM_DV_ASMC/PUTM_DV_ASMC.kicad_sch (KiCad schematic)
At the start: 0 parts

Commit message: after review2
Other:
- sheet Connectors ports: added none; removed ADC, GPIO
- sheet Microcontroller ports: added none; removed ADC, GPIO
Changed lines of the file:
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@@
-	(wire
-		(pts
-			(xy 144.78 109.22) (xy 237.49 109.22)
-		)
-		(stroke
-			(width 0)
-			(type default)
-		)
-	)
 	(wire
 		(pts
@@
 		(pts
 			(xy 210.82 91.44) (xy 237.49 91.44)
-		)
-		(stroke
-			(width 0)
-			(type default)
-		)
-	)
-	(wire
-		(pts
-			(xy 144.78 111.76) (xy 237.49 111.76)
 		)
 		(stroke
@@
 			)
 		)
-		(pin "ADC" bidirectional
-			(at 237.49 109.22 180)
-			(effects
-				(font
-					(size 1.27 1.27)
-				)
-				(justify left)
-			)
-		)
-		(pin "GPIO" bidirectional
-			(at 237.49 111.76 180)
-			(effects
-				(font
-					(size 1.27 1.27)
-				)
-				(justify left)
-			)
-		)
 		(pin "ODRIVE[1..4]" input
 			(at 237.49 60.96 180)
@@
 			(effects
 				(font
-					(size 1.27 1.27)
-				)
-				(justify right)
-			)
-		)
-		(pin "ADC" bidirectional
-			(at 144.78 109.22 0)
-			(effects
-				(font
-					(size 1.27 1.27)
-				)
-				(justify right)
-			)
-		)
-		(pin "GPIO" bidirectional
-			(at 144.78 111.76 0)
-			(effects
-				(font
