File: hardware/PUTM_DV_ASMC/Odrive_power_supply.kicad_sch (KiCad schematic)
At the start: 24 parts, among them IC1 BTS722204ESAXUMA1

Commit message: update spi schema
Connections:
- net NSS renamed CSN1
Changed lines of the file:
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@@
 		)
 	)
-	(hierarchical_label "NSS"
+	(hierarchical_label "CSN1"
 		(shape input)
 		(at 99.06 91.44 180)

Commit message: update pcb layout after rewiev
Other:
- note added: "1* 0 [Ohm] or 330 [Ohm]"
- note removed: "1* 1k2 to 330R - daisy chain"
Changed lines of the file:
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@@
 		)
 	)
-	(text "1* 1k2 to 330R - daisy chain"
+	(text "1* 0 [Ohm] or 330 [Ohm]"
 		(exclude_from_sim no)
 		(at 205.74 132.08 0)
